Commit message: Changes

File: example_2/description/ros2_control/diffbot.ros2_control.xacro (robot description, xacro)
@@ -1,4 +1,5 @@
 <?xml version="1.0"?>
 <robot xmlns:xacro="http://www.ros.org/wiki/xacro">
+  <!-- Drive system (wheels) -->
   <xacro:macro name="diffbot_ros2_control" params="name prefix use_mock_hardware">
     <ros2_control name="${name}" type="system">
@@ -34,3 +35,47 @@
     </ros2_control>
   </xacro:macro>
+  <!-- Actuation system (legs) -->
+  <xacro:macro name="actuation_ros2_control" params="name prefix use_mock_hardware">
+    <ros2_control name="${name}" type="system">
+      <xacro:unless value="${use_mock_hardware}">
+        <hardware>
+          <plugin>ros2_control_demo_example_2/ActuationSystemHardware</plugin>
+          <param name="act0_serial_num">527103</param>
+          <param name="act0_port_num">0</param>
+          <param name="act1_serial_num">527103</param>
+          <param name="act1_port_num">1</param>
+          <param name="act2_serial_num">527164</param>
+          <param name="act2_port_num">0</param>
+          <param name="act3_serial_num">527164</param>
+          <param name="act3_port_num">1</param>
+        </hardware>
+      </xacro:unless>
+      <xacro:if value="${use_mock_hardware}">
+        <hardware>
+          <plugin>mock_components/GenericSystem</plugin>
+          <param name="calculate_dynamics">true</param>
+        </hardware>
+      </xacro:if>
+      <joint name="${prefix}actuator_joint_0">
+        <command_interface name="velocity"/>
+        <state_interface name="position"/>
+        <state_interface name="velocity"/>
+      </joint>
+      <joint name="${prefix}actuator_joint_1">
+        <command_interface name="velocity"/>
+        <state_interface name="position"/>
+        <state_interface name="velocity"/>
+      </joint>
+      <joint name="${prefix}actuator_joint_2">
+        <command_interface name="velocity"/>
+        <state_interface name="position"/>
+        <state_interface name="velocity"/>
+      </joint>
+      <joint name="${prefix}actuator_joint_3">
+        <command_interface name="velocity"/>
+        <state_interface name="position"/>
+        <state_interface name="velocity"/>
+      </joint>
+    </ros2_control>
+  </xacro:macro>
 </robot>

File: example_2/description/urdf/diffbot.urdf copy.xacro (robot description, xacro)
@@ -25,3 +25,8 @@
     prefix="$(arg prefix)"
     use_mock_hardware="$(arg use_mock_hardware)"/>
+  <!-- Instantiate actuation system -->
+  <xacro:actuation_ros2_control
+    name="ActuationSystem"
+    prefix="$(arg prefix)"
+    use_mock_hardware="$(arg use_mock_hardware)"/>
 </robot>
