Commit message: Wokring SLAM on robot

File: robot_description/urdf/ibex_core.urdf.xacro (robot description, xacro)
@@ -79,4 +79,58 @@
         <origin xyz="0 0 ${wheel_radius - (base_height / 2.0)}" rpy="0 0 0"/>
     </joint>
+    <link name="imu_link">
+        <inertial>
+            <origin xyz="-0.00552433659106688 0.000168210391520346 0.000514000497342681" rpy="0 0 0" />
+            <mass value="0.000528415362211671" />
+            <inertia ixx="1.46176048428261E-08" ixy="1.40015117949421E-10" ixz="-1.99633872937403E-12"
+                    iyy="8.59662482954888E-09" iyz="7.52375112767959E-12"
+                    izz="2.30279421279312E-08" />
+        </inertial>
+        <visual>
+            <origin xyz="0 0 0" rpy="0 0 0" />
+            <geometry>
+                <box size="0.1 0.1 0.05"/>
+            </geometry>
+            <material name="blue" />
+        </visual>
+        <collision>
+            <origin xyz="0 0 0" rpy="0 0 0" />
+            <geometry>
+                <box size="0.1 0.1 0.05"/>
+            </geometry>
+        </collision>
+    </link>
+    <joint name="imu_joint" type="fixed">
+        <origin xyz="0.45 -0.30 0.07" rpy="0 0 0" />
+        <parent link="base_link" />
+        <child link="imu_link" />
+    </joint>
+    <link name="laser">
+        <inertial>
+            <origin xyz="-0.011945780406062 -0.000381929217680526 -0.0170649378129477" rpy="0 0 0" />
+            <mass value="0.073084435549317" />
+            <inertia ixx="1.96074931730795E-05" ixy="-3.62091076640009E-07" ixz="4.28230084046735E-07"
+                    iyy="2.40983835136327E-05" iyz="1.50180909250652E-08"
+                    izz="4.14184164228595E-05" />
+        </inertial>
+        <visual>
+            <origin xyz="0 0 0" rpy="0 0 0" />
+            <geometry>
+            <cylinder radius="0.035" length="0.05"/>
+            </geometry>
+            <material name="blue"/>
+        </visual>
+        <collision>
+            <origin xyz="0 0 0" rpy="0 0 0" />
+            <geometry>
+            <cylinder radius="0.035" length="0.05"/>
+            </geometry>
+        </collision>
+    </link>
+    <joint name="laser_joint" type="fixed">
+        <origin xyz="0.45 0 0.12" rpy="0 0 0" />
+        <parent link="base_link" />
+        <child link="laser" />
+    </joint>
     <xacro:wheel_macro name_prefix="rear_right"
                         x_offset="${-wheel_axle_x_offset}"

Commit message: Lidar working with og robot

File: robot_description/urdf/ibex_core.urdf.xacro (robot description, xacro)
@@ -79,4 +79,58 @@
         <origin xyz="0 0 ${wheel_radius - (base_height / 2.0)}" rpy="0 0 0"/>
     </joint>
+        <link name="imu_link">
+        <inertial>
+            <origin xyz="-0.00552433659106688 0.000168210391520346 0.000514000497342681" rpy="0 0 0" />
+            <mass value="0.000528415362211671" />
+            <inertia ixx="1.46176048428261E-08" ixy="1.40015117949421E-10" ixz="-1.99633872937403E-12"
+                    iyy="8.59662482954888E-09" iyz="7.52375112767959E-12"
+                    izz="2.30279421279312E-08" />
+        </inertial>
+        <visual>
+            <origin xyz="0 0 0" rpy="0 0 0" />
+            <geometry>
+                <box size="0.1 0.1 0.05"/>
+            </geometry>
+            <material name="blue" />
+        </visual>
+        <collision>
+            <origin xyz="0 0 0" rpy="0 0 0" />
+            <geometry>
+                <box size="0.1 0.1 0.05"/>
+            </geometry>
+        </collision>
+    </link>
+    <joint name="imu_joint" type="fixed">
+        <origin xyz="0.45 -0.30 0.07" rpy="0 0 0" />
+        <parent link="base_link" />
+        <child link="imu_link" />
+    </joint>
+    <link name="laser">
+        <inertial>
+            <origin xyz="-0.011945780406062 -0.000381929217680526 -0.0170649378129477" rpy="0 0 0" />
+            <mass value="0.073084435549317" />
+            <inertia ixx="1.96074931730795E-05" ixy="-3.62091076640009E-07" ixz="4.28230084046735E-07"
+                    iyy="2.40983835136327E-05" iyz="1.50180909250652E-08"
+                    izz="4.14184164228595E-05" />
+        </inertial>
+        <visual>
+            <origin xyz="0 0 0" rpy="0 0 0" />
+            <geometry>
+            <cylinder radius="0.035" length="0.05"/>
+            </geometry>
+            <material name="blue"/>
+        </visual>
+        <collision>
+            <origin xyz="0 0 0" rpy="0 0 0" />
+            <geometry>
+            <cylinder radius="0.035" length="0.05"/>
+            </geometry>
+        </collision>
+    </link>
+    <joint name="laser_joint" type="fixed">
+        <origin xyz="0.45 0 0.12" rpy="0 0 0" />
+        <parent link="base_link" />
+        <child link="laser" />
+    </joint>
     <xacro:wheel_macro name_prefix="rear_right"
                         x_offset="${-wheel_axle_x_offset}"

File: robot_description/urdf/ibex_ros2_control.urdf.xacro (robot description, xacro)
@@ -2,9 +2,9 @@
 <robot xmlns:xacro="http://www.ros.org/wiki/xacro" name="ibex">
   <ros2_control name="IbexDiffDirve" type="system">
-      <!-- <hardware>
+      <hardware>
         <plugin>mock_components/GenericSystem</plugin>
         <param name="calculate_dynamics">true</param>
-      </hardware> -->
-      <hardware>
+      </hardware>
+      <!-- <hardware>
         <plugin>ibex_control/DiffBotSystemHardware</plugin>
         <param name="bl_serial_num">527103</param>
@@ -16,5 +16,5 @@
         <param name="fr_serial_num">527164</param>
         <param name="fr_port_num">3</param>
-      </hardware>
+      </hardware> -->
       <joint name="front_left_wheel_joint">
         <command_interface name="velocity">

File: robot_sim_description/urdf/ibex_core.urdf.xacro (robot description, xacro)
@@ -79,4 +79,60 @@
         <origin xyz="0 0 ${wheel_radius - (base_height / 2.0)}" rpy="0 0 0"/>
     </joint>
+        <link name="imu_link">
+        <inertial>
+            <origin xyz="-0.00552433659106688 0.000168210391520346 0.000514000497342681" rpy="0 0 0" />
+            <mass value="0.000528415362211671" />
+            <inertia ixx="1.46176048428261E-08" ixy="1.40015117949421E-10" ixz="-1.99633872937403E-12"
+                    iyy="8.59662482954888E-09" iyz="7.52375112767959E-12"
+                    izz="2.30279421279312E-08" />
+        </inertial>
+        <visual>
+            <origin xyz="0 0 0" rpy="0 0 0" />
+            <geometry>
+                <box size="0.1 0.1 0.05"/>
+            </geometry>
+            <material name="blue" />
+        </visual>
+        <collision>
+            <origin xyz="0 0 0" rpy="0 0 0" />
+            <geometry>
+                <box size="0.1 0.1 0.05"/>
+            </geometry>
+        </collision>
+    </link>
+    <joint name="imu_joint" type="fixed">
+        <origin xyz="0 0 0.0698986241758014" rpy="0 0 0" />
+        <parent link="base_link" />
+        <child link="imu_link" />
+        <axis xyz="0 0 0" />
+    </joint>
+    <link name="laser_link">
+        <inertial>
+            <origin xyz="-0.011945780406062 -0.000381929217680526 -0.0170649378129477" rpy="0 0 0" />
+            <mass value="0.073084435549317" />
+            <inertia ixx="1.96074931730795E-05" ixy="-3.62091076640009E-07" ixz="4.28230084046735E-07"
+                    iyy="2.40983835136327E-05" iyz="1.50180909250652E-08"
+                    izz="4.14184164228595E-05" />
+        </inertial>
+        <visual>
+            <origin xyz="0 0 0" rpy="0 0 0" />
+            <geometry>
+            <cylinder radius="0.035" length="0.05"/>
+            </geometry>
+            <material name="blue"/>
+        </visual>
+        <collision>
+            <origin xyz="0 0 0" rpy="0 0 0" />
+            <geometry>
+            <cylinder radius="0.035" length="0.05"/>
+            </geometry>
+        </collision>
+    </link>
+    <joint name="laser_joint" type="fixed">
+        <origin xyz="-0.0050526 -0.0023221 0.1208" rpy="0 0 3.14" />
+        <parent link="base_link" />
+        <child link="laser_link" />
+        <axis xyz="0 0 0" />
+    </joint>
     <xacro:wheel_macro name_prefix="rear_right"
                         x_offset="${-wheel_axle_x_offset}"

File: robot_sim_description/urdf/ibex_gazebo.urdf.xacro (robot description, xacro)
@@ -6,3 +6,52 @@
     </plugin>
     </gazebo>
+        <gazebo>
+        <plugin filename="gz-sim-sensors-system" name="gz::sim::systems::Sensors">
+            <render_engine>ogre2</render_engine>
+        </plugin>
+    </gazebo>
+    <!-- <gazebo>
+        <plugin filename="gz-sim-imu-system" name="gz::sim::systems::Imu">
+        </plugin>
+        <plugin filename="gz-sim-sensors-system" name="gz::sim::systems::Sensors">
+            <render_engine>ogre2</render_engine>
+        </plugin>
+    </gazebo> -->
+    <gazebo reference="imu_link">
+        <sensor name="imu_sensor" type="imu">
+            <topic>imu/out</topic>
+            <always_on>true</always_on>
+            <update_rate>100</update_rate>
+            <plugin filename="gz-sim-imu-system" name="gz::sim::systems::Imu"/>
+        </sensor>
+    </gazebo>
+    <gazebo reference="laser_link">
+        <sensor name="lidar" type="gpu_lidar">
+        <always_on>true</always_on>
+        <visualize>true</visualize>
+        <topic>scan</topic>
+        <update_rate>5</update_rate>
+        <gz_frame_id>laser_link</gz_frame_id>
+        <lidar>
+            <scan>
+            <horizontal>
+                <samples>360</samples>
+                <resolution>1.00000</resolution>
+                <min_angle>0.000000</min_angle>
+                <max_angle>6.280000</max_angle>
+            </horizontal>
+            </scan>
+            <range>
+            <min>0.120000</min>
+            <max>12.0</max>
+            <resolution>0.02</resolution>
+            </range>
+            <noise>
+            <type>gaussian</type>
+            <mean>0.0</mean>
+            <stddev>0.01</stddev>
+            </noise>
+        </lidar>
+        </sensor>
+    </gazebo>
 </robot>
