Commit message: Position contrl (not working)

File: robot_description/urdf/ibex_actuation_ros2_control.urdf.xacro (robot description, xacro)
@@ -1,5 +1,5 @@
 <?xml version="1.0"?>
 <robot xmlns:xacro="http://www.ros.org/wiki/xacro" name="ibex">
-  <ros2_control name="IbexDiffDirve" type="system">
+  <ros2_control name="IbexActuation" type="system">
       <!-- <hardware>
         <plugin>mock_components/GenericSystem</plugin>

File: robot_description/urdf/ibex_core.urdf.xacro (robot description, xacro)
@@ -146,5 +146,5 @@
                 <box size="0.1 0.1 0.05"/>
             </geometry>
-            <material name="blue" />
+            <material name="black" />
         </visual>
         <collision>
@@ -173,5 +173,5 @@
             <cylinder radius="0.035" length="0.05"/>
             </geometry>
-            <material name="blue"/>
+            <material name="black"/>
         </visual>
         <collision>
