Commit message: Working lidar on urdf

File: install/robot_sim_description/share/robot_sim_description/urdf/ibex_core.urdf.xacro (robot description, xacro)
@@ -79,24 +79,24 @@
         <origin xyz="0 0 ${wheel_radius - (base_height / 2.0)}" rpy="0 0 0"/>
     </joint>
-    <!-- <link name="imu_link">
+    <link name="imu_link">
         <inertial>
-        <origin xyz="-0.00552433659106688 0.000168210391520346 0.000514000497342681" rpy="0 0 0" />
-        <mass value="0.000528415362211671" />
-        <inertia ixx="1.46176048428261E-08" ixy="1.40015117949421E-10" ixz="-1.99633872937403E-12"
-                iyy="8.59662482954888E-09" iyz="7.52375112767959E-12"
-                izz="2.30279421279312E-08" />
+            <origin xyz="-0.00552433659106688 0.000168210391520346 0.000514000497342681" rpy="0 0 0" />
+            <mass value="0.000528415362211671" />
+            <inertia ixx="1.46176048428261E-08" ixy="1.40015117949421E-10" ixz="-1.99633872937403E-12"
+                    iyy="8.59662482954888E-09" iyz="7.52375112767959E-12"
+                    izz="2.30279421279312E-08" />
         </inertial>
         <visual>
-        <origin xyz="0 0 0" rpy="0 0 0" />
-        <geometry>
-            <mesh filename="package://robot_sim_description/meshes/imu_link.STL" />
-        </geometry>
-        <material name="blue"/>
+            <origin xyz="0 0 0" rpy="0 0 0" />
+            <geometry>
+                <box size="0.1 0.1 0.05"/>
+            </geometry>
+            <material name="blue" />
         </visual>
         <collision>
-        <origin xyz="0 0 0" rpy="0 0 0" />
-        <geometry>
-            <mesh filename="package://robot_sim_description/meshes/imu_link.STL" />
-        </geometry>
+            <origin xyz="0 0 0" rpy="0 0 0" />
+            <geometry>
+                <box size="0.1 0.1 0.05"/>
+            </geometry>
         </collision>
     </link>
@@ -106,5 +106,33 @@
         <child link="imu_link" />
         <axis xyz="0 0 0" />
-    </joint> -->
+    </joint>
+    <link name="laser_link">
+        <inertial>
+            <origin xyz="-0.011945780406062 -0.000381929217680526 -0.0170649378129477" rpy="0 0 0" />
+            <mass value="0.073084435549317" />
+            <inertia ixx="1.96074931730795E-05" ixy="-3.62091076640009E-07" ixz="4.28230084046735E-07"
+                    iyy="2.40983835136327E-05" iyz="1.50180909250652E-08"
+                    izz="4.14184164228595E-05" />
+        </inertial>
+        <visual>
+            <origin xyz="0 0 0" rpy="0 0 0" />
+            <geometry>
+            <cylinder radius="0.035" length="0.05"/>
+            </geometry>
+            <material name="dark_grey"/>
+        </visual>
+        <collision>
+            <origin xyz="0 0 0" rpy="0 0 0" />
+            <geometry>
+            <cylinder radius="0.035" length="0.05"/>
+            </geometry>
+        </collision>
+    </link>
+    <joint name="laser_joint" type="fixed">
+        <origin xyz="-0.0050526 -0.0023221 0.1208" rpy="0 0 3.14" />
+        <parent link="base_link" />
+        <child link="laser_link" />
+        <axis xyz="0 0 0" />
+    </joint>
     <xacro:wheel_macro name_prefix="rear_right"
                         x_offset="${-wheel_axle_x_offset}"

File: install/robot_sim_description/share/robot_sim_description/urdf/ibex_gazebo.urdf.xacro (robot description, xacro)
@@ -6,5 +6,5 @@
     </plugin>
     </gazebo>
-    <!-- <gazebo>
+    <gazebo>
         <plugin filename="gz-sim-imu-system" name="gz::sim::systems::Imu">
         </plugin>
@@ -41,4 +41,4 @@
         </lidar>
         </sensor>
-    </gazebo> -->
+    </gazebo>
 </robot>

Commit message: Working with slam toolbox

File: install/robot_sim_description/share/robot_sim_description/urdf/ibex_core.urdf.xacro (robot description, xacro)
@@ -120,5 +120,5 @@
             <cylinder radius="0.035" length="0.05"/>
             </geometry>
-            <material name="dark_grey"/>
+            <material name="blue"/>
         </visual>
         <collision>
