Commit message: New URDF broken

File: miguel_urdf/urdf/cad_urdf_gazebo.urdf.xacro (robot description, xacro)
@@ -1,4 +1,4 @@
 <?xml version="1.0"?>
-<robot xmlns:xacro="http://www.ros.org/wiki/xacro" name="ibex">
+<robot xmlns:xacro="http://www.ros.org/wiki/xacro" name="cad_urdf">
     <gazebo>
     <plugin filename="gz_ros2_control-system" name="gz_ros2_control::GazeboSimROS2ControlPlugin">

File: robot_description/urdf/ibex_core.urdf.xacro (robot description, xacro)
@@ -66,5 +66,5 @@
                 <origin xyz="0 0 0" rpy="${pi / 2.0} 0 0" />
             </collision>
-    </link>
+        </link>
             <joint name="${name_prefix}_wheel_joint" type="continuous">
         <parent link="base_link" />
