Commit message: Fix collision

File: robot_sim_description/urdf/cad_urdf_core.urdf.xacro (robot description, xacro)
@@ -14,8 +14,21 @@
     <!-- Mesh scale -->
     <xacro:property name="mesh_scale"               value="0.001 0.001 0.001" />
-    <xacro:property name="wheel_mass" value="3.321118377201799"/>
-    <xacro:property name="wheel_ixx"  value="0.017539"/>
-    <xacro:property name="wheel_iyy"  value="0.011505"/>
-    <xacro:property name="wheel_izz"  value="0.012355"/>
+    <xacro:property name="chassis_mass" value="5.0" />
+    <xacro:property name="wheel_mass" value="0.5" />
+    <xacro:property name="wheel_radius" value="0.102" />
+    <xacro:property name="wheel_thickness" value="0.069" />
+    <xacro:property name="chassis_length"   value="0.4096"/>   <!-- 2 ft -->
+    <xacro:property name="chassis_width"    value="0.9144"/>   <!-- 2 ft -->
+    <xacro:property name="chassis_height"   value="0.0762"/>   <!-- 6 in -->
+    <xacro:property name="wheel_offset_x" value="0.2794"/>
+    <xacro:property name="wheel_offset_y" value="0.2708"/>
+    <xacro:property name="wheel_offset_z" value="0.0516"/>
+    <xacro:property name="mesh_rpy"       value="0 0 -1.57079"/>
+    <xacro:property name="wheel_ixx" value="${(wheel_mass/12.0) * (3*wheel_radius*wheel_radius + wheel_thickness*wheel_thickness)}"/>
+    <xacro:property name="wheel_iyy" value="${(wheel_mass/2.0)  * (wheel_radius*wheel_radius)}"/>
+    <xacro:property name="wheel_izz" value="${wheel_ixx}"/>
+    <xacro:property name="chassis_ixx" value="${(chassis_mass / 12.0) * (chassis_height*chassis_height + chassis_width*chassis_width)}"/>
+    <xacro:property name="chassis_iyy" value="${(chassis_mass / 12.0) * (chassis_length*chassis_length + chassis_height*chassis_height)}"/>
+    <xacro:property name="chassis_izz" value="${(chassis_mass / 12.0) * (chassis_length*chassis_length + chassis_width*chassis_width)}"/>
     <xacro:property name="wheel_com_x_abs" value="0.08445"/>
     <xacro:property name="wheel_com_y"     value="-0.003338577608035853"/>
@@ -63,7 +76,5 @@
                 <origin xyz="${wheel_com_x_abs * inertial_x_mult} ${wheel_com_y} ${wheel_com_z}" rpy="0 0 0"/>
                 <mass value="${wheel_mass}"/>
-                <inertia ixx="${wheel_ixx}" iyy="${wheel_iyy}" izz="${wheel_izz}"
-                         ixy="0.0" iyz="0.0" ixz="0.0"/>
-            </inertial>
+                <inertia ixx="${wheel_ixx}" iyy="${wheel_iyy}" izz="${wheel_izz}" ixy="0" iyz="0" ixz="0"/> </inertial>
             <visual>
                 <origin xyz="${origin_xyz}" rpy="${origin_rpy}"/>
@@ -74,7 +85,7 @@
             </visual>
             <collision>
-                <origin xyz="${origin_xyz}" rpy="${origin_rpy}"/>
-                <geometry>
-                    <mesh filename="${mesh_file}" scale="${mesh_scale}"/>
+                <origin xyz="0 0 0" rpy="1.57079 0 0"/>  <!-- Rotate 90° to align with wheel axis -->
+                <geometry>
+                    <cylinder radius="${wheel_radius}" length="${wheel_thickness}"/>
                 </geometry>
             </collision>
@@ -91,9 +102,9 @@
         <inertial>
             <origin xyz="-2.1660968987257366e-16 -1.7328775189805893e-16 0.028711464160038225" rpy="0 0 0"/>
-            <mass value="26.36828818920337"/>
-            <inertia ixx="2.061838" iyy="1.248081" izz="3.230816" ixy="-0.0" iyz="0.0" ixz="-0.0"/>
+            <mass value="${chassis_mass}"/>
+            <inertia ixx="${chassis_ixx}" iyy="${chassis_iyy}" izz="${chassis_izz}" ixy="0" iyz="0" ixz="0"/>
         </inertial>
         <visual>
-            <origin xyz="0 0 0" rpy="0 0 -1.57079"/>
+            <origin xyz="0 0 0" rpy="${mesh_rpy}"/>
             <geometry>
                 <mesh filename="${mesh_base_link}" scale="${mesh_scale}"/>
@@ -102,7 +113,7 @@
         </visual>
         <collision>
-            <origin xyz="0 0 0" rpy="0 0 -1.57079"/>
+            <origin xyz="0 0 ${chassis_height / 2.0}" rpy="${mesh_rpy}"/>  <!-- Center at half height -->
             <geometry>
-                <mesh filename="${mesh_base_link}" scale="${mesh_scale}"/>
+                <box size="${chassis_length} ${chassis_width} ${chassis_height}"/>
             </geometry>
         </collision>
@@ -113,5 +124,43 @@
         <origin xyz="0 0 0.0484" rpy="0 0 0"/>
     </joint>
-    <!-- Flipper and Wheel Links using Macros -->
+    <!-- Wheels     -->
+    <xacro:wheel_macro
+        name="front_left"
+        mesh_file="${mesh_front_left_wheel}"
+        origin_xyz="-${wheel_offset_x} -${wheel_offset_y} -${wheel_offset_z}"
+        origin_rpy="${mesh_rpy}"
+        inertial_x_mult="-1"
+        joint_origin_xyz="${wheel_offset_x} ${wheel_offset_y} ${wheel_offset_z}"
+        joint_origin_rpy="0 0 0"
+        joint_axis="0.0 1.0 0.0" />
+    <xacro:wheel_macro
+        name="front_right"
+        mesh_file="${mesh_front_right_wheel}"
+        origin_xyz="-${wheel_offset_x} ${wheel_offset_y} -${wheel_offset_z}"
+        origin_rpy="${mesh_rpy}"
+        inertial_x_mult="1"
+        joint_origin_xyz="${wheel_offset_x} -${wheel_offset_y} ${wheel_offset_z}"
+        joint_origin_rpy="0 0 0"
+        joint_axis="0.0 1.0 0.0" />
+    <xacro:wheel_macro
+        name="rear_left"
+        mesh_file="${mesh_rear_left_wheel}"
+        origin_xyz="${wheel_offset_x} -${wheel_offset_y} -${wheel_offset_z}"
+        origin_rpy="${mesh_rpy}"
+        inertial_x_mult="-1"
+        joint_origin_xyz="-${wheel_offset_x} ${wheel_offset_y} ${wheel_offset_z}"
+        joint_origin_rpy="0 0 0"
+        joint_axis="0.0 1.0 0.0" />
+    <xacro:wheel_macro
+        name="rear_right"
+        mesh_file="${mesh_rear_right_wheel}"
+        origin_xyz="${wheel_offset_x} ${wheel_offset_y} -${wheel_offset_z}"
+        origin_rpy="${mesh_rpy}"
+        inertial_x_mult="1"
+        joint_origin_xyz="-${wheel_offset_x} -${wheel_offset_y} ${wheel_offset_z}"
+        joint_origin_rpy="0 0 0"
+        joint_axis="0.0 1.0 0.0" />
+</robot>
+        <!-- Flipper and Wheel Links using Macros -->
     <!-- <xacro:flipper_macro
         name="front_left_flipper"
@@ -174,41 +223,4 @@
         joint_origin_xyz="-0.3108 -0.2794 0.0516"
         joint_origin_rpy="0 0 0" /> -->
-    <!-- Wheels     -->
-    <xacro:wheel_macro
-        name="front_left"
-        mesh_file="${mesh_front_left_wheel}"
-        origin_xyz="-0.2794 -0.2708 -0.0516"
-        origin_rpy="0 0 -1.57079"
-        inertial_x_mult="-1"
-        joint_origin_xyz="0.2794 0.2708 0.0516"
-        joint_origin_rpy="0 0 0"
-        joint_axis="0.0 1.0 0.0" />
-    <xacro:wheel_macro
-        name="front_right"
-        mesh_file="${mesh_front_right_wheel}"
-        origin_xyz="-0.2794 0.2708 -0.0516"
-        origin_rpy="0 0 -1.57079"
-        inertial_x_mult="1"
-        joint_origin_xyz=" 0.2794 -0.2708 0.0516"
-        joint_origin_rpy="0 0 0"
-        joint_axis="0.0 1.0 0.0" />
-    <xacro:wheel_macro
-        name="rear_left"
-        mesh_file="${mesh_rear_left_wheel}"
-        origin_xyz=" 0.2794 -0.2708 -0.0516"
-        origin_rpy="0 0 -1.57079"
-        inertial_x_mult="-1"
-        joint_origin_xyz="-0.2794 0.2708 0.0516"
-        joint_origin_rpy="0 0 0"
-        joint_axis="0.0 1.0 0.0" />
-    <xacro:wheel_macro
-        name="rear_right"
-        mesh_file="${mesh_rear_right_wheel}"
-        origin_xyz="0.2794 0.2708 -0.0516"
-        origin_rpy="0 0 -1.57079"
-        inertial_x_mult="1"
-        joint_origin_xyz="-0.2794 -0.2708 0.0516"
-        joint_origin_rpy="0 0 0"
-        joint_axis="0.0 1.0 0.0" />
     <!-- <xacro:wheel_macro
         name="front_left_wheel"
@@ -247,3 +259,2 @@
         joint_origin_rpy="0 0 0"
         joint_axis="-1.0 0.0 0.0" /> -->
-</robot>

File: robot_sim_description/urdf/cad_urdf_ros2_control.urdf.xacro (robot description, xacro)
@@ -9,6 +9,6 @@
         <joint name="front_left_wheel_joint">
           <command_interface name="velocity">
-            <param name="min">-1</param>
-            <param name="max">1</param>
+            <param name="min">-10</param>
+            <param name="max">10</param>
           </command_interface>
           <state_interface name="position"/>
@@ -18,6 +18,6 @@
         <joint name="front_right_wheel_joint">
           <command_interface name="velocity">
-            <param name="min">-1</param>
-            <param name="max">1</param>
+            <param name="min">-10</param>
+            <param name="max">10</param>
           </command_interface>
           <state_interface name="position"/>
@@ -27,6 +27,6 @@
         <joint name="rear_left_wheel_joint">
           <command_interface name="velocity">
-            <param name="min">-1</param>
-            <param name="max">1</param>
+            <param name="min">-10</param>
+            <param name="max">10</param>
           </command_interface>
           <state_interface name="position"/>
@@ -36,6 +36,6 @@
         <joint name="rear_right_wheel_joint">
           <command_interface name="velocity">
-            <param name="min">-1</param>
-            <param name="max">1</param>
+            <param name="min">-10</param>
+            <param name="max">10</param>
           </command_interface>
           <state_interface name="position"/>

Commit message: I added flippers

File: robot_sim_description/urdf/cad_urdf_core.urdf.xacro (robot description, xacro)
@@ -8,8 +8,8 @@
     <xacro:property name="mesh_rear_left_wheel"     value="${base_file_path}wheel_rear_left.stl" />
     <xacro:property name="mesh_rear_right_wheel"    value="${base_file_path}wheel_rear_right.stl" />
-    <!-- <xacro:property name="mesh_front_left_flipper"  value="${base_file_path}flipper_front_left.stl" /> -->
-    <!-- <xacro:property name="mesh_front_right_flipper" value="${base_file_path}flipper_front_right.stl" /> -->
-    <!-- <xacro:property name="mesh_rear_left_flipper"   value="${base_file_path}flipper_rear_left.stl" /> -->
-    <!-- <xacro:property name="mesh_rear_right_flipper"  value="${base_file_path}flipper_rear_right.stl" /> -->
+    <xacro:property name="mesh_front_left_flipper"  value="${base_file_path}flipper_front_left.stl" />
+    <xacro:property name="mesh_front_right_flipper" value="${base_file_path}flipper_front_right.stl" />
+    <xacro:property name="mesh_rear_left_flipper"   value="${base_file_path}flipper_front_left.stl" />
+    <xacro:property name="mesh_rear_right_flipper"  value="${base_file_path}flipper_rear_right.stl" />
     <!-- Mesh scale -->
     <xacro:property name="mesh_scale"               value="0.001 0.001 0.001" />
@@ -39,5 +39,5 @@
     <link name="base_footprint" />
     <!-- Flipper Macro with Fixed Joint -->
-    <!-- <xacro:macro name="flipper_macro" params="name mesh_file origin_xyz origin_rpy inertial_origin_xyz inertial_mass inertial_ixx inertial_iyy inertial_izz inertial_ixy inertial_iyz inertial_ixz joint_origin_xyz joint_origin_rpy">
+    <xacro:macro name="flipper_macro" params="name mesh_file origin_xyz origin_rpy inertial_origin_xyz inertial_mass inertial_ixx inertial_iyy inertial_izz inertial_ixy inertial_iyz inertial_ixz joint_origin_xyz joint_origin_rpy">
         <link name="${name}">
             <inertial>
@@ -66,5 +66,5 @@
             <child link="${name}"/>
         </joint>
-    </xacro:macro> -->
+    </xacro:macro>
     <!-- Wheel Macro with Continuous Joint -->
     <xacro:macro name="wheel_macro" params="name_prefix x_offset y_offset z_offset">
@@ -143,7 +143,6 @@
                         y_offset="${-wheel_offset_y}"
                         z_offset="${wheel_offset_z}" />
-</robot>
-        <!-- Flipper and Wheel Links using Macros -->
-    <!-- <xacro:flipper_macro
+            <!-- Flipper and Wheel Links using Macros -->
+    <xacro:flipper_macro
         name="front_left_flipper"
         mesh_file="${mesh_front_left_flipper}"
@@ -151,5 +150,5 @@
         origin_rpy="0 0 -1.57079"
         inertial_origin_xyz="0.044450000334023076 0.005646153366949069 0.249739430595357"
-        inertial_mass="7.296846138774613"
+        inertial_mass="0.01"
         inertial_ixx="0.281827"
         inertial_iyy="0.262219"
@@ -166,5 +165,5 @@
         origin_rpy="0 0 -1.57079"
         inertial_origin_xyz="0.044450000334053885 0.01614155751815055 0.24928119135390578"
-        inertial_mass="7.296846138774627"
+        inertial_mass="0.01"
         inertial_ixx="0.281827"
         inertial_iyy="0.256055"
@@ -175,11 +174,12 @@
         joint_origin_xyz="0.3108 -0.2794 0.0516"
         joint_origin_rpy="0 0 0" />
+<!-- bad one -->
     <xacro:flipper_macro
         name="rear_left_flipper"
         mesh_file="${mesh_rear_left_flipper}"
-        origin_xyz="0.3108 -0.2794 -0.0516"
+        origin_xyz="0.3108 0.4294 -0.0516"
         origin_rpy="0 0 -1.57079"
         inertial_origin_xyz="-0.044450000334023076 0.22872695820013356 0.10042729128305261"
-        inertial_mass="7.29684613877462"
+        inertial_mass="0.01"
         inertial_ixx="0.281827"
         inertial_iyy="0.100275"
@@ -196,5 +196,5 @@
         origin_rpy="0 0 -1.57079"
         inertial_origin_xyz="-0.044450000334023076 0.016141557518147776 0.24928119135391122"
-        inertial_mass="7.29684613877462"
+        inertial_mass="0.01"
         inertial_ixx="0.281827"
         inertial_iyy="0.256055"
@@ -204,5 +204,6 @@
         inertial_ixz="0.0"
         joint_origin_xyz="-0.3108 -0.2794 0.0516"
-        joint_origin_rpy="0 0 0" /> -->
+        joint_origin_rpy="0 0 0" />
+</robot>
     <!-- <xacro:wheel_macro
         name="front_left_wheel"

Commit message: Added cave world
motion kinda sucks on the rocky terrain
unsure if that is a configurable thing
or sim is running poorly on my laptop

File: robot_sim_description/urdf/cad_urdf_core.urdf.xacro (robot description, xacro)
@@ -139,5 +139,5 @@
                 <box size="0.1 0.1 0.05"/>
             </geometry>
-            <material name="blue" />
+            <material name="black" />
         </visual>
         <collision>
@@ -167,5 +167,5 @@
             <cylinder radius="0.035" length="0.05"/>
             </geometry>
-            <material name="blue"/>
+            <material name="black"/>
         </visual>
         <collision>

Commit message: Recommiting bags using Git LFS

File: robot_sim_description/urdf/cad_urdf_core.urdf.xacro (robot description, xacro)
@@ -177,8 +177,7 @@
     </link>
     <joint name="laser_joint" type="fixed">
-        <origin xyz="-0.0050526 -0.0023221 0.1208" rpy="0 0 3.14" />
-        <parent link="base_link" />
-        <child link="laser_link" />
-        <axis xyz="0 0 0" />
+        <origin xyz="0.50 0 0.05" rpy="0 0 0"/>
+        <parent link="base_link"/>
+        <child link="laser_link"/>
     </joint>
     <!-- Wheels     -->
